File: ChipigniteExplain.kicad_pcb (KiCad board)
At the start: 4 copper layers, 53.5 x 65.5 mm, 251 parts, among them J1 Conn_01x02, J10 Conn_01x02, J11 Conn_01x06, J2 Conn_01x02, J3 Conn_01x03, J4 USB_C, J5 613012243121, J6 613012243121, J7 Conn_02x03_Odd_Even, Q1 DMN2005K, SW1 434121025816, SW2 434121025816, SW3 434121025816, SW4 434121025816, SW5 434121025816, SW6 193-8MSR, U1 TLV1117LV33, U2 TPD1E05U06QDPYRQ1, U3 157112V12700, U4 RP2040, U5 W25Q32JVSS, U6 AP2112K-1.2, U7 ICE40UP5K-SG48ITR, X1 24MHz, Y1 12.0MHz

Commit message: BOM MPN additions and tweaks
Parts:
- U7: value ICE40UP5K-SG48ITR -> ICE40UP5K-SG48I
